File: preamp.brd (EAGLE design)
At the start: 16 x 25 mm, 19 parts, among them Q1 SST201, Q2 SST201, Q3 SST201

Commit message: Change gain resistor to match IRL, add TODO notes
Parts:
- R3: value 500k -> 1k
Changed lines of the file:
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@@
 <?xml version="1.0" encoding="utf-8"?>
 <!DOCTYPE eagle SYSTEM "eagle.dtd">
-<eagle version="9.2.2">
+<eagle version="9.2.1">
 <drawing>
 <settings>
@@
 <attribute name="VALUE" x="15.54" y="6.53" size="1.27" layer="27" rot="R90"/>
 </element>
-<element name="R3" library="rcl" package="R1206" value="500k" x="3.6" y="7.1" smashed="yes">
+<element name="R3" library="rcl" package="R1206" value="1k" x="3.6" y="7.1" smashed="yes">
 <attribute name="VALUE" x="2.33" y="4.56" size="1.27" layer="27"/>
 </element>
