File: 3-3/preamp.sch (EAGLE design)
At the start: 23 parts, among them Q1 SST201, Q2 SST201, Q3 SST201

Commit message: Base 3-3 after 1-1 after building 2-2
Parts:
- removed C4, C5: DNP, rcl:C-EUC1206
- removed POT1, POT2: (no value), wirepad:3,17/1,3
- R3: value 500 -> 510R
Connections:
- removed net N$2: POT1.P, R3.1, SJ1.2
- net GND: now also R3.1; no longer C4.1, C5.1, POT2.P
- net N$3: no longer C4.2
- net N$7: no longer C5.2
- net PZ-1: now also SJ1.2
Other:
- moved on the sheet: PZ-1, PZ-GND, R1, R2, R5, R6, SJ1, XLR1
